File: Skin-Sensor/V0/Skin_Sensor_Modular.kicad_pcb (KiCad board)
At the start: 2 copper layers, 51.8 x 23.9 mm, 142 parts, among them J1 JTAGICE3-10p, SW1 SW_PUSH, U1 ADP7102, U2 ATSAMD21E18A, U3 USB2, U4 LSM9DS1, U5 LP5521YQ, U6 DPS310, U7 DPS310, X1 ABS06

Commit message: Skin Sensor Dump
Other:
- board text added: "Alt. Pressure Sensors"
- board text added: "Inertial Measurement Unit"
- board text added: "Pressure Sensors"
- board text added: "Programmer Module"
- board text added: "Sensor Node"
- board text added: "Status LED"
Changed lines of the file:
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@@
     (links 235)
     (no_connects 7)
-    (area 78.595 48.794999 133.38 113.701231)
+    (area 69.142858 83.025 147.021429 115.85)
     (thickness 1.6)
-    (drawings 170)
+    (drawings 176)
     (tracks 866)
     (zones 0)
@@
       (net 98 "Net-(U7-Pad5)"))
   )
+  (gr_text "Status LED" (at 116.6 114.5) (layer F.Fab)
+    (effects (font (size 1.5 1.5) (thickness 0.3)))
+  )
+  (gr_text "Inertial\nMeasurement\nUnit" (at 139.7 99.1) (layer F.Fab)
+    (effects (font (size 1.5 1.5) (thickness 0.3)))
+  )
+  (gr_text "Programmer\nModule" (at 117.3 85.5) (layer F.Fab)
+    (effects (font (size 1.5 1.5) (thickness 0.3)))
+  )
+  (gr_text "Sensor Node" (at 99.6 85.8) (layer F.Fab)
+    (effects (font (size 1.5 1.5) (thickness 0.3)))
+  )
+  (gr_text "Alt.\nPressure\nSensors" (at 74 105.4) (layer F.Fab)
+    (effects (font (size 1.5 1.5) (thickness 0.3)))
+  )
+  (gr_text "Pressure\nSensors" (at 74.2 93.9) (layer F.Fab)
+    (effects (font (size 1.5 1.5) (thickness 0.3)))
+  )
   (gr_line (start 121.8031 93.85) (end 121.8031 96.5) (angle 90) (layer Edge.Cuts) (width 0.1))
