File: Skin-Sensor/V1/Skin-Sensor-V1.sch (KiCad schematic (older format))
At the start: 68 parts, among them J1 JTAGICE3-10p, SW1 SW_PUSH, U1 ADP7102, U2 ATSAMD21E18A, U3 USB2, U4 LSM9DS1, U5 LP5521YQ, U6 DPS310, U7 DPS310, X1 ABS06

Commit message: Skin Sensor Dump
Parts:
- removed SW1: SW_PUSH, _Fab_Footprint:SPST-NO-TL3700, symbol SW_PUSH-RESCUE-LPS25H
- removed U2: ATSAMD21E18A, _Fab_Footprint:QFN-32-1EP_5x5mm_Pitch0.5mm, symbol ATSAMD21E18A
- added U?: ATSAMD21E18A, symbol ATSAMD21E18A
Connections:
- wire segments 498 -> 614
Other:
- note added: "4-Pin FFC \nI2C Bus"
- note added: "6-Pin FFC \nIntermodule Network"
- note added: "Alt. Pressure Sensors"
- note added: "Connector To Programmer Addon"
- note added: "FFC Connector"
- note added: "Inertial Measurement Unit"
- note added: "JTAG Header"
- note added: "Pressure Sensors"
- note added: "SENSOR NODE"
- note added: "Sensor Bus Pullup Resistors (I2C)"
- note added: "Sensors"
- note added: "USB"
- note removed: "Avoid pins 3,5,6,11-14,21,24"
- note removed: "MAIN MODULE"
- note removed: "NB: USB is 22/23 on R-Series"
- note removed: "R-Series Compatibility:"
- note removed: "Testing A New Sensor"
- moved on the sheet: C1, C10, C11, C12, C13, C14, C15, C16, C17, C18, C19, C2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
