File: Skin-Sensor/V1/hw/Skin-Sensor-V1.kicad_pcb (KiCad board)
At the start: 2 copper layers, 57.8 x 23.1 mm, 116 parts, among them J1 JTAGICE3-10p, SW1 SW_PUSH, U1 ADP7102, U2 ATSAMD21E18A, U3 USB2, U4 LSM9DS1, U5 LP5521YQ, U6 DPS310, U7 DPS310, X1 ABS06

Commit message: V1 rev, in all its glory
Parts:
- removed C10, C36: 100nF, Capacitors_SMD:C_0402
- removed C11: sj2, _Fab_Footprint:SJ-2-1-no
- removed C12: sj1, _Fab_Footprint:SJ-2-1-no
- removed C13, C14: WM1386x04, _Fab_Footprint:WM1386x04-REC
- removed C29, C34: WM1386x06, _Fab_Footprint:WM1387x06-REC
- removed C35: 4.7UF, Capacitors_SMD:C_0402
- removed L1, L2: LPS25H, _Fab_Footprint:LPS25H
- removed R4, R5, R6, R7: 10k, Resistors_SMD:R_0402
- removed the REF** at (88.9, 98.0)
- removed the REF** at (112.6, 100.3)
- removed the REF** at (112.6, 99.9)
- removed the REF** at (112.6, 99.5)
- removed the REF** at (112.6, 99.1)
- removed the REF** at (115.8, 100.4)
- removed the REF** at (116.3, 100.4)
- removed the REF** at (116.7, 100.4)
- removed the REF** at (117.2, 100.4)
- removed the REF** at (117.6, 100.4)
- removed the REF** at (118.1, 100.4)
- removed the REF** at (88.9, 98.5)
- removed the REF** at (118.5, 100.4)
- removed the REF** at (118.5, 101.3)
- removed the REF** at (118.1, 101.3)
- removed the REF** at (117.7, 101.3)
- removed the REF** at (117.2, 101.3)
- removed the REF** at (116.8, 101.3)
- removed the REF** at (116.3, 101.3)
- removed the REF** at (112.6, 98.7)
- removed the REF** at (115.8, 101.3)
- removed the REF** at (121.7, 100.2)
- removed the REF** at (88.9, 98.8)
- removed the REF** at (121.7, 99.8)
- removed the REF** at (121.7, 99.4)
- removed the REF** at (121.7, 99.0)
- removed the REF** at (121.7, 98.6)
- removed the REF** at (121.7, 98.2)
- removed the REF** at (121.7, 97.8)
- removed the REF** at (121.7, 97.4)
- removed the REF** at (121.7, 97.0)
- removed the REF** at (122.7, 100.2)
- removed the REF** at (122.7, 99.8)
- removed the REF** at (88.9, 99.2)
- removed the REF** at (122.7, 99.5)
- removed the REF** at (122.7, 99.0)
- removed the REF** at (122.7, 98.7)
- removed the REF** at (122.7, 98.2)
- removed the REF** at (122.7, 97.8)
- removed the REF** at (122.7, 97.5)
- removed the REF** at (122.7, 97.0)
- removed the REF** at (129.1, 103.3)
- removed the REF** at (129.1, 93.3)
- removed the REF** at (111.0, 98.8)
- removed the REF** at (111.0, 99.2)
- removed the REF** at (111.0, 99.6)
- removed the REF** at (111.0, 100.0)
- removed the REF** at (111.0, 100.4)
- added C4: WM1386x10, _CSL:WM1387x10-REC, F.Cu at (110.1, 89.9)
- added REF**: Pin_Header_Straight_1x01_Pitch2.00mm, Pin_Headers:Pin_Header_Straight_1x01_Pitch2.00mm, F.Cu at (118.1, 105.0)
- added REF**: BreakawayHole, _CSL:BreakawayHole, F.Cu at (109.6, 94.2)
- added REF**: BreakawayHole, _CSL:BreakawayHole, F.Cu at (109.2, 93.7)
- added REF**: BreakawayHole, _CSL:BreakawayHole, F.Cu at (108.8, 93.3)
- added REF**: BreakawayHole, _CSL:BreakawayHole, F.Cu at (109.4, 91.8)
- added REF**: BreakawayHole, _CSL:BreakawayHole, F.Cu at (110.7, 93.1)
- added REF**: BreakawayHole, _CSL:BreakawayHole, F.Cu at (110.3, 92.7)
- added REF**: BreakawayHole, _CSL:BreakawayHole, F.Cu at (109.8, 92.2)
- added REF**: BreakawayHole, _CSL:BreakawayHole, F.Cu at (109.0, 91.4)
- added REF**: BreakawayHole, _CSL:BreakawayHole, F.Cu at (107.3, 89.7)
- added REF**: BreakawayHole, _CSL:BreakawayHole, F.Cu at (108.6, 91.0)
- added REF**: Pin_Header_Straight_1x01_Pitch2.00mm, Pin_Headers:Pin_Header_Straight_1x01_Pitch2.00mm, F.Cu at (118.1, 95.0)
- added REF**: BreakawayHole, _CSL:BreakawayHole, F.Cu at (108.2, 90.6)
- added REF**: BreakawayHole, _CSL:BreakawayHole, F.Cu at (107.7, 90.1)
- added REF**: BreakawayHole, _CSL:BreakawayHole, F.Cu at (106.9, 89.3)
- added REF**: BreakawayHole, _CSL:BreakawayHole, F.Cu at (99.4, 89.2)
- added REF**: BreakawayHole, _CSL:BreakawayHole, F.Cu at (100.0, 89.2)
- added REF**: BreakawayHole, _CSL:BreakawayHole, F.Cu at (100.6, 89.1)
- added REF**: BreakawayHole, _CSL:BreakawayHole, F.Cu at (98.8, 89.2)
- added REF**: BreakawayHole, _CSL:BreakawayHole, F.Cu at (101.2, 89.1)
- added REF**: BreakawayHole, _CSL:BreakawayHole, F.Cu at (100.6, 87.9)
- added REF**: BreakawayHole, _CSL:BreakawayHole, F.Cu at (101.2, 87.8)
- added REF**: BreakawayHole, _CSL:BreakawayHole, F.Cu at (106.3, 90.8)
- added REF**: BreakawayHole, _CSL:BreakawayHole, F.Cu at (99.4, 87.8)
- added REF**: BreakawayHole, _CSL:BreakawayHole, F.Cu at (100.0, 87.8)
- added REF**: BreakawayHole, _CSL:BreakawayHole, F.Cu at (98.8, 87.8)
- added REF**: BreakawayHole, _CSL:BreakawayHole, F.Cu at (112.2, 98.8)
- added REF**: BreakawayHole, _CSL:BreakawayHole, F.Cu at (112.2, 101.2)
- added REF**: BreakawayHole, _CSL:BreakawayHole, F.Cu at (112.2, 100.0)
- added REF**: BreakawayHole, _CSL:BreakawayHole, F.Cu at (112.2, 99.4)
- added REF**: BreakawayHole, _CSL:BreakawayHole, F.Cu at (112.2, 100.6)
- added REF**: BreakawayHole, _CSL:BreakawayHole, F.Cu at (110.9, 99.4)
- added REF**: BreakawayHole, _CSL:BreakawayHole, F.Cu at (110.9, 101.2)
- added REF**: BreakawayHole, _CSL:BreakawayHole, F.Cu at (107.5, 92.1)
- added REF**: BreakawayHole, _CSL:BreakawayHole, F.Cu at (110.9, 100.6)
- added REF**: BreakawayHole, _CSL:BreakawayHole, F.Cu at (110.9, 98.8)
- added REF**: BreakawayHole, _CSL:BreakawayHole, F.Cu at (110.9, 100.0)
- added REF**: BreakawayHole, _CSL:BreakawayHole, F.Cu at (98.8, 110.9)
- added REF**: BreakawayHole, _CSL:BreakawayHole, F.Cu at (99.4, 110.9)
- added REF**: BreakawayHole, _CSL:BreakawayHole, F.Cu at (100.0, 110.8)
- added REF**: BreakawayHole, _CSL:BreakawayHole, F.Cu at (101.2, 110.8)
- added REF**: BreakawayHole, _CSL:BreakawayHole, F.Cu at (100.6, 110.8)
- added REF**: BreakawayHole, _CSL:BreakawayHole, F.Cu at (101.2, 112.2)
- added REF**: BreakawayHole, _CSL:BreakawayHole, F.Cu at (98.8, 112.2)
- added REF**: BreakawayHole, _CSL:BreakawayHole, F.Cu at (108.4, 92.9)
- added REF**: BreakawayHole, _CSL:BreakawayHole, F.Cu at (100.6, 112.2)
- added REF**: BreakawayHole, _CSL:BreakawayHole, F.Cu at (99.4, 112.2)
- added REF**: BreakawayHole, _CSL:BreakawayHole, F.Cu at (100.0, 112.2)
- added REF**: BreakawayHole, _CSL:BreakawayHole, F.Cu at (87.8, 101.2)
- added REF**: BreakawayHole, _CSL:BreakawayHole, F.Cu at (87.8, 99.4)
- added REF**: BreakawayHole, _CSL:BreakawayHole, F.Cu at (87.8, 98.8)
- added REF**: BreakawayHole, _CSL:BreakawayHole, F.Cu at (87.8, 100.0)
- added REF**: BreakawayHole, _CSL:BreakawayHole, F.Cu at (87.8, 100.6)
- added REF**: BreakawayHole, _CSL:BreakawayHole, F.Cu at (89.2, 101.2)
- added REF**: BreakawayHole, _CSL:BreakawayHole, F.Cu at (89.2, 100.6)
- added REF**: BreakawayHole, _CSL:BreakawayHole, F.Cu at (107.9, 92.5)
- added REF**: BreakawayHole, _CSL:BreakawayHole, F.Cu at (89.2, 98.8)
- added REF**: BreakawayHole, _CSL:BreakawayHole, F.Cu at (89.2, 100.0)
- added REF**: BreakawayHole, _CSL:BreakawayHole, F.Cu at (89.2, 99.4)
- added REF**: BreakawayHole, _CSL:BreakawayHole, F.Cu at (106.7, 91.2)
- added REF**: BreakawayHole, _CSL:BreakawayHole, F.Cu at (107.1, 91.6)
- added REF**: BreakawayHole, _CSL:BreakawayHole, F.Cu at (105.8, 90.4)
- added SW2: SW_PUSH, _Fab_Footprint:4-PLCC, B.Cu at (110.1, 89.9)
- C19, C20, C21, C22, C23: moved to F.Cu
- C9: value 4.7UF -> WM1386x10; footprint Capacitors_SMD:C_0402 -> _CSL:WM1387x10-REC
- SW1: footprint _Fab_Footprint:SPST-NO-TL3700 -> _Fab_Footprint:4-PLCC
- moved C24 41.1 mm to (78.5, 102.1), turned to 270 degrees
- moved R13 39.7 mm to (78.5, 100.2), turned to 270 degrees
- moved C27 38.5 mm to (78.5, 98.5), turned to 90 degrees
- moved R12 37.5 mm to (82.7, 103.3), turned to 0 degrees
- moved D2 36.4 mm to (81.2, 100.0), turned to 90 degrees
- moved U5 36.4 mm to (81.2, 100.0), turned to 0 degrees
- moved C26 35.4 mm to (80.2, 96.8), turned to 0 degrees
- moved C25 33.0 mm to (82.2, 96.8), turned to 0 degrees
- moved C39 31.3 mm to (86.0, 100.0), turned to 90 degrees
- moved U6 27.3 mm to (100.8, 85.0)
- moved C3 27.2 mm to (101.5, 83.8), turned to 324 degrees
- moved R14 26.6 mm to (97.9, 85.4), turned to 108 degrees
- moved C38 26.5 mm to (100.0, 86.0)
- moved C28 26.1 mm to (98.5, 83.8), turned to 36 degrees
- moved C41 25.1 mm to (101.5, 116.2), turned to 216 degrees
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Connections:
- C15 pad 1: S5GND -> GND
- C15 pad 2: S5SCL -> SCL
- C15 pad 3: S5SDA -> SDA
- C15 pad 4: S5VCC -> +3V3
- C15 pad 5: S5GND -> GND
- C19 pad 1: S5VCC -> +3V3
- C20 pad 1: S5VCC -> +3V3
- C21 pad 1: S5VCC -> +3V3
- C24 pad 1: S6VCC -> +3V3
- C24 pad 2: S6GND -> GND
- C25 pad 2: S6GND -> GND
- C28 pad 1: S3GND -> GND
- C28 pad 2: S3VCC -> +3V3
- C3 pad 1: S3VCC -> +3V3
- C3 pad 2: S3GND -> GND
- C37 pad 1: S4GND -> GND
- C37 pad 2: S4SCL -> SCL
- C37 pad 3: S4SDA -> SDA
- C37 pad 4: S4VCC -> +3V3
- C37 pad 5: S4GND -> GND
- C38 pad 1: S3GND -> GND
- C38 pad 2: S3SCL -> SCL
- C38 pad 3: S3SDA -> SDA
- C38 pad 4: S3VCC -> +3V3
- C38 pad 5: S3GND -> GND
- C39 pad 1: S6GND -> GND
- C39 pad 2: S6SCL -> SCL
- C39 pad 3: S6SDA -> SDA
- C39 pad 4: S6VCC -> +3V3
- C39 pad 5: S6GND -> GND
- C40 pad 1: S4VCC -> +3V3
- C40 pad 2: S4GND -> GND
- C41 pad 1: S4GND -> GND
- C41 pad 2: S4VCC -> +3V3
- C9 pad 1: S1VCC -> GND
- C9 pad 2: S1GND -> D-
- D2 pad 4: S6GND -> GND
- J1 pad 1: DP/SWCLK -> PVCC
- J1 pad 10: (no net) -> PRESET
- J1 pad 2: PGND -> PSWDIO
- J1 pad 3: (no net) -> PGND
- J1 pad 4: PVCC -> PSWCLK
- J1 pad 5: DM/SWDIO -> (no net)
- J1 pad 6: PRESET -> (no net)
- R10 pad 1: S5VCC -> +3V3
- R11 pad 1: S5VCC -> +3V3
- R12 pad 1: S6VCC -> +3V3
- R13 pad 1: S6VCC -> +3V3
- R14 pad 2: S3GND -> GND
- R8 pad 1: S5VCC -> +3V3
- R9 pad 1: S5VCC -> +3V3
- U3 pad 2: DM/SWDIO -> PD-
- U3 pad 3: DP/SWCLK -> PD+
- U4 pad 1: S5VCC -> +3V3
- U4 pad 2: S5SCL -> SCL
- U4 pad 22: S5VCC -> +3V3
- U4 pad 23: S5VCC -> +3V3
- U4 pad 3: S5VCC -> +3V3
- U4 pad 4: S5SDA -> SDA
- U5 pad 13: S6SDA -> SDA
- U5 pad 15: S6SCL -> SCL
- U5 pad 20: S6GND -> GND
- U5 pad 21: S6GND -> GND
- U5 pad 25: S6GND -> GND
- U5 pad 3: S6VCC -> +3V3
- U5 pad 4: S6GND -> GND
- U5 pad 5: S6GND -> GND
- U5 pad 7: S6GND -> GND
- U6 pad 1: S3GND -> GND
- U6 pad 3: S3SDA -> SDA
- U6 pad 4: S3SCL -> SCL
- U6 pad 6: S3VCC -> +3V3
- U6 pad 7: S3GND -> GND
- U6 pad 8: S3VCC -> +3V3
- U7 pad 1: S4GND -> GND
- U7 pad 3: S4SDA -> SDA
- U7 pad 4: S4SCL -> SCL
- U7 pad 6: S4VCC -> +3V3
- U7 pad 7: S4GND -> GND
- U7 pad 8: S4VCC -> +3V3
Routing:
- net GND: track 65.5 -> 162.3 mm, vias 0 -> 17
- net +3V3: track 79.8 -> 159.7 mm, vias 5 -> 13
- net SCL: track 40.6 -> 81.6 mm, vias 4 -> 6
- net SDA: track 37.7 -> 77.6 mm, vias 4 -> 8
- net S6GND: track 26.8 -> 0.00 mm, vias 2 -> 0
- net S2GND: track 21.7 -> 0.00 mm, vias 1 -> 0
- net S5VCC: track 20.4 -> 0.00 mm, vias 1 -> 0
- net S6VCC: track 18.8 -> 0.00 mm, vias 2 -> 0
- net S3GND: track 18.3 -> 0.00 mm, vias 3 -> 0
- net S1GND: track 17.7 -> 0.00 mm, vias 2 -> 0
- net S1VCC: track 16.1 -> 0.00 mm, vias 2 -> 0
- net S4GND: track 14.4 -> 0.00 mm, vias 1 -> 0
- net S6SDA: track 9.50 -> 0.00 mm
- net DM/SWDIO: track 8.97 -> 0.00 mm, vias 1 -> 0
- net S2VCC: track 8.81 -> 0.00 mm, vias 1 -> 0
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- removed copper zone on B.Cu, net S2GND
- removed copper zone on F.Cu, net S2GND
Other:
- board size 57.8 x 23.1 mm -> 161.4 x 51.1 mm
- rule trace_min: 0.127 -> 0.06
- board text added: "0x76"
- board text added: "0x77"
- board text removed: "JTAG"
- board text removed: "USB"
