File: Skin-Sensor/V1/hw/Skin-Sensor-V1.sch (KiCad schematic (older format))
At the start: 67 parts, among them J1 JTAGICE3-10p, U1 ADP7102, U3 USB2, U4 LSM9DS1, U5 LP5521YQ, U6 DPS310, U7 DPS310, X1 ABS06

Commit message: V1 rev, in all its glory
Parts:
- removed C10, C36: 100nF, Capacitors_SMD:C_0402, symbol CAP
- removed C11: sj2, _Fab_Footprint:SJ-2-1-no, symbol solder_jumper_2_1_no_conn
- removed C12: sj1, _Fab_Footprint:SJ-2-1-no, symbol solder_jumper_2_1_no_conn
- removed C13, C14: WM1386x04, _Fab_Footprint:WM1386x04-REC, symbol WM1386x04
- removed C29, C34: WM1386x06, _Fab_Footprint:WM1387x06-REC, symbol WM1386x06
- removed C35, C9: 4.7UF, Capacitors_SMD:C_0402, symbol CAP
- removed L1, L2: LPS25H, _Fab_Footprint:LPS25H, symbol LPS25H
- removed R4, R5, R6, R7: 10k, Resistors_SMD:R_0402, symbol RES
- added C4, C9: WM1386x10, _CSL:WM1387x10-REC, symbol WM1386x10
- added SW1, SW2: SW_PUSH, _Fab_Footprint:4-PLCC, symbol SW_PUSH
- U2: renamed from U?; footprint (none) -> _Fab_Footprint:QFN-32-1EP_5x5mm_Pitch0.5mm
Connections:
- net S3GND is gone; now on net GND: C28.1, C3.2, C38.1, C38.5, R14.2, U6.1 (GND), U6.7 (GND)
- net S3SCL is gone; now on net SCL: C38.2, U6.4 (SCK)
- net S3SDA is gone; now on net SDA: C38.3, U6.3 (SDI)
- net S3VCC is gone; now on net +3V3: C28.2, C3.1, C38.4, U6.6 (VDDIO), U6.8 (VDD)
- net S4GND is gone; now on net GND: C37.1, C37.5, C40.2, C41.1, U7.1 (GND), U7.7 (GND)
- net S4SCL is gone; now on net SCL: C37.2, U7.4 (SCK)
- net S4SDA is gone; now on net SDA: C37.3, U7.3 (SDI)
- net S4VCC is gone; now on net +3V3: C37.4, C40.1, C41.2, U7.6 (VDDIO), U7.8 (VDD)
- net S5SCL is gone; now on net SCL: C15.2, U4.2 (SCL/SPC)
- net S5SDA is gone; now on net SDA: C15.3, U4.4 (SDA/SDI/SDO)
- net S5VCC is gone; now on net +3V3: C15.4, C19.1, C20.1, C21.1, R10.1, R11.1, R8.1, R9.1, U4.1 (VDDIO), U4.22 (VDD), U4.23 (VDD), U4.3 (VDDIO)
- net S6GND is gone; now on net GND: C24.2, C25.2, C39.1, C39.5, D2.4 (COMMON_CATHODE), U5.20 (ASEL0), U5.21 (ASEL1), U5.25 (GND), U5.4 (GND), U5.5 (CLK_32K), U5.7 (TRIG)
- net S6SCL is gone; now on net SCL: C39.2, U5.15 (SCL)
- net S6SDA is gone; now on net SDA: C39.3, U5.13 (SDA)
- net S6VCC is gone; now on net +3V3: C24.1, C39.4, R12.1, R13.1, U5.3 (VDD)
- net +3V3: now also C9.9
- net D+: now also C9.3
- net D-: now also C9.2
- net GND: now also C15.1, C15.5, C9.1, C9.10, C9.11, SW1.1, SW1.2
- net PGND: now also C4.1, C4.10, C4.11, SW2.1, SW2.2
- net PRESET: now also C4.4, SW2.3, SW2.4
- net PVCC: now also C4.2
- net PVRAW: now also C4.3
- net RESET: now also C9.7, SW1.3, SW1.4
- net S5GND: no longer C15.1, C15.5
- net SWCLK: now also C9.4
- net SWDIO: now also C9.5, C9.6
- net VRAW: now also C9.8
- net DM/SWDIO renamed PD-
- net PD-: now also C4.9; no longer J1.2 (SWDIO)
- net DP/SWCLK renamed PD+
- net PD+: now also C4.8; no longer J1.4 (SWDCLK)
- new net PSWCLK: C4.7, J1.4 (SWDCLK)
- new net PSWDIO: C4.5, C4.6, J1.2 (SWDIO)
Other:
- note added: "4-Pin FFC \nI2C Bus"
- note added: "6-Pin FFC \nIntermodule Network"
- note added: "Connector To Programmer Addon"
- note added: "FFC Connector"
- note added: "Inertial Measurement Unit"
- note added: "JTAG Header"
- note added: "Pressure Sensors"
- note added: "SENSOR NODE"
- note added: "Sensor Bus Pullup Resistors (I2C)"
- note added: "Sensors"
- note added: "USB"
- note removed: "Avoid pins 3,5,6,11-14,21,24"
- note removed: "I2C Addr: 0x5c"
- note removed: "I2C Addr: 0x5d"
- note removed: "MAIN MODULE"
- note removed: "NB: USB is 22/23 on R-Series"
- note removed: "R-Series Compatibility:"
- note removed: "Testing A New Sensor"
- moved on the sheet: C1, C15, C16, C17, C18, C19, C2, C20, C21, C22, C23, C24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
